Commit message: Tuned laserscan intertia and fixed laserscan rang

File: urdf/warehouse_bot_sim.gazebo.xacro (robot description, xacro)
@@ -6,5 +6,4 @@
   </gazebo>
   <!-- Wheel Properties -->
-  <!-- TODO: check out fdir1 properties  -->
   <gazebo reference="wheel_left_link">
     <mu1>2000</mu1>
@@ -74,5 +73,5 @@
           <horizontal>
             <samples>541</samples>
-            <resolution>0.005817</resolution>
+            <resolution>1</resolution>
             <min_angle>-1.57</min_angle>
             <max_angle>1.57</max_angle>

File: urdf/warehouse_bot_sim.urdf.xacro (robot description, xacro)
@@ -53,7 +53,7 @@
     </visual>
     <inertial>
-      <origin xyz="0 0 0"/>
+      <origin xyz="-0.169 0 0"/>
       <mass value="0.003"/>
-      <inertia ixx="0.001" ixy="0.0" ixz="0.0" iyy="0.001" iyz="0.0" izz="0.001"/>
+      <inertia ixx="0.0000012" ixy="0.0" ixz="0.0" iyy="0.0000012" iyz="0.0" izz="0.0000012"/>
     </inertial>
   </link>
