Commit message: Added in xacro macro for the caster wheel

File: urdf/warehouse_bot_sim.urdf.xacro (robot description, xacro)
@@ -2,4 +2,33 @@
 <robot name="warehouse_bot"
   xmlns:xacro="http://ros.org/wiki/xacro">
+  <xacro:macro name="caster" params="name *origin">
+    <link name="${name}_link">
+      <visual>
+        <origin xyz="0 0 0" rpy="0 0 0"/>
+        <geometry>
+          <sphere radius="0.015"/>
+        </geometry>
+        <material name="grey">
+          <color rgba="0.5 0.5 0.5 1.0"/>
+        </material>
+      </visual>
+      <collision>
+        <origin xyz="0 0 0" rpy="0 0 0"/>
+        <geometry>
+          <sphere radius="0.015"/>
+        </geometry>
+      </collision>
+      <inertial>
+        <origin xyz="0 0 0"/>
+        <mass value="0.003"/>
+        <inertia ixx="0.001" ixy="0.0" ixz="0.0" iyy="0.001" iyz="0.0" izz="0.001"/>
+      </inertial>
+    </link>
+    <joint name="${name}_joint" type="fixed">
+      <parent link="base_link"/>
+      <child link="${name}_link"/>
+      <xacro:insert_block name="origin"/>
+    </joint>
+  </xacro:macro>
   <link name="base_laser">
     <visual>
@@ -44,5 +73,5 @@
     <origin xyz="0.0 0.0 0.05"/>
   </joint>`
-  <joint name="wheel_left_joint" type="fixed">
+  <joint name="wheel_left_joint" type="continuous">
     <parent link="base_link"/>
     <child link="wheel_left_link"/>
@@ -61,3 +90,6 @@
     <origin xyz="0.169 0.0 0.035856" rpy="3.142 0.0 0.0"/>
   </joint>
+  <xacro:caster name="caster_top_left">
+    <origin xyz="0.18 0.18 -0.035" rpy="0.0 0.0 0.0"/>
+  </xacro:caster>
 </robot>

Commit message: Added in all caster wheels

File: urdf/warehouse_bot_sim.urdf.xacro (robot description, xacro)
@@ -31,4 +31,16 @@
     </joint>
   </xacro:macro>
+  <xacro:caster name="caster_top_left">
+    <origin xyz="0.16 0.16 -0.035" rpy="0.0 0.0 0.0"/>
+  </xacro:caster>
+  <xacro:caster name="caster_bottom_left">
+    <origin xyz="-0.16 0.16 -0.035" rpy="0.0 0.0 0.0"/>
+  </xacro:caster>
+  <xacro:caster name="caster_bottom_right">
+    <origin xyz="-0.16 -0.16 -0.035" rpy="0.0 0.0 0.0"/>
+  </xacro:caster>
+  <xacro:caster name="caster_top_right">
+    <origin xyz="0.16 -0.16 -0.035" rpy="0.0 0.0 0.0"/>
+  </xacro:caster>
   <link name="base_laser">
     <visual>
@@ -90,6 +102,3 @@
     <origin xyz="0.169 0.0 0.035856" rpy="3.142 0.0 0.0"/>
   </joint>
-  <xacro:caster name="caster_top_left">
-    <origin xyz="0.18 0.18 -0.035" rpy="0.0 0.0 0.0"/>
-  </xacro:caster>
 </robot>

Commit message: Added in intertia and collision tags

File: urdf/warehouse_bot_sim.urdf.xacro (robot description, xacro)
@@ -2,5 +2,5 @@
 <robot name="warehouse_bot"
   xmlns:xacro="http://ros.org/wiki/xacro">
-<xacro:include filename="$(find warehousebot_simulation)/urdf/warehouse_bot_sim.gazebo.xacro"/>
+  <xacro:include filename="$(find warehousebot_simulation)/urdf/warehouse_bot_sim.gazebo.xacro"/>
   <xacro:macro name="caster" params="name *origin">
     <link name="${name}_link">
@@ -60,4 +60,15 @@
       <origin rpy="0 0 0" xyz="0 0 0"/>
     </visual>
+    <collision name="base_collision">
+      <geometry>
+        <mesh filename="package://warehousebot_simulation/meshes/left_wheel.stl" scale="0.01 0.01 0.01"/>
+      </geometry>
+      <origin rpy="0 0 0" xyz="0 0 0"/>
+    </collision>
+    <inertial>
+      <origin xyz="0 0 0"/>
+      <mass value="1"/>
+      <inertia ixx="0.00282485" ixy="-1.41127e-06" ixz="1.32139e-08" iyy="0.00283002" iyz="2.09836e-07" izz="0.00515906"/>
+    </inertial>
   </link>
   <link name="wheel_right_link">
@@ -68,4 +79,15 @@
       <origin rpy="0 0 0" xyz="0 0 0"/>
     </visual>
+    <collision name="base_collision">
+      <geometry>
+        <mesh filename="package://warehousebot_simulation/meshes/right_wheel.stl" scale="0.01 0.01 0.01"/>
+      </geometry>
+      <origin rpy="0 0 0" xyz="0 0 0"/>
+    </collision>
+    <inertial>
+      <origin xyz="0 0 0"/>
+      <mass value="1"/>
+      <inertia ixx="0.00282485" ixy="-1.41127e-06" ixz="1.32139e-08" iyy="0.00283002" iyz="2.09836e-07" izz="0.00515906"/>
+    </inertial>
   </link>
   <link name="base_footprint"/>
@@ -80,4 +102,15 @@
       <origin rpy="0 0 0" xyz="0 0 0"/>
     </visual>
+    <collision name="base_collision">
+      <geometry>
+        <mesh filename="package://warehousebot_simulation/meshes/bot_chassis.stl" scale="0.01 0.01 0.01"/>
+      </geometry>
+      <origin rpy="0 0 0" xyz="0 0 0"/>
+    </collision>
+    <inertial>
+      <mass value="80"/>
+      <origin rpy="0 0 0" xyz="0 0 0"/>
+      <inertia ixx="5.44729" ixy="0.00186274" ixz="0.901373" iyy="6.17857" iyz="-0.0011154" izz="3.76947"/>
+    </inertial>
   </link>
   <joint name="base_footprint_to_base_link" type="fixed">

Commit message: changed interia to be a sphere for robot base

File: urdf/warehouse_bot_sim.urdf.xacro (robot description, xacro)
@@ -109,7 +109,7 @@
     </collision>
     <inertial>
-      <mass value="80"/>
-      <origin rpy="0 0 0" xyz="0 0 0"/>
-      <inertia ixx="5.44729" ixy="0.00186274" ixz="0.901373" iyy="6.17857" iyz="-0.0011154" izz="3.76947"/>
+      <mass value="550"/>
+      <origin rpy="0 0 0" xyz="0 0 0 "/>
+      <inertia ixx="220" ixy="0" ixz="0" iyy="220" iyz="0" izz="220"/>
     </inertial>
   </link>

Commit message: Added in inertial tag for the laser scan

File: urdf/warehouse_bot_sim.urdf.xacro (robot description, xacro)
@@ -52,4 +52,9 @@
       <origin rpy="0 0 0" xyz="0 0 0"/>
     </visual>
+    <inertial>
+      <origin xyz="0 0 0"/>
+      <mass value="0.003"/>
+      <inertia ixx="0.001" ixy="0.0" ixz="0.0" iyy="0.001" iyz="0.0" izz="0.001"/>
+    </inertial>
   </link>
   <link name="wheel_left_link">
@@ -60,9 +65,9 @@
       <origin rpy="0 0 0" xyz="0 0 0"/>
     </visual>
-    <collision name="base_collision">
+    <collision>
+      <origin xyz="0 0 0" rpy="0 0 0"/>
       <geometry>
-        <mesh filename="package://warehousebot_simulation/meshes/left_wheel.stl" scale="0.01 0.01 0.01"/>
+        <cylinder length="0.018" radius="0.033"/>
       </geometry>
-      <origin rpy="0 0 0" xyz="0 0 0"/>
     </collision>
     <inertial>
@@ -79,9 +84,9 @@
       <origin rpy="0 0 0" xyz="0 0 0"/>
     </visual>
-    <collision name="base_collision">
+    <collision>
+      <origin xyz="0 0 0" rpy="0 0 0"/>
       <geometry>
-        <mesh filename="package://warehousebot_simulation/meshes/right_wheel.stl" scale="0.01 0.01 0.01"/>
+        <cylinder length="0.018" radius="0.033"/>
       </geometry>
-      <origin rpy="0 0 0" xyz="0 0 0"/>
     </collision>
     <inertial>

Commit message: fixed incorrect intertia values

File: urdf/warehouse_bot_sim.urdf.xacro (robot description, xacro)
@@ -114,7 +114,7 @@
     </collision>
     <inertial>
-      <mass value="550"/>
+      <mass value="20"/>
       <origin rpy="0 0 0" xyz="0 0 0 "/>
-      <inertia ixx="220" ixy="0" ixz="0" iyy="220" iyz="0" izz="220"/>
+      <inertia ixx="0.32" ixy="0" ixz="0" iyy="0.32" iyz="0" izz="0.32"/>
     </inertial>
   </link>

Commit message: fixed collision issues for wheels

File: urdf/warehouse_bot_sim.urdf.xacro (robot description, xacro)
@@ -68,5 +68,5 @@
       <origin xyz="0 0 0" rpy="0 0 0"/>
       <geometry>
-        <cylinder length="0.018" radius="0.033"/>
+        <cylinder length="0.05" radius="0.0985"/>
       </geometry>
     </collision>
@@ -87,5 +87,5 @@
       <origin xyz="0 0 0" rpy="0 0 0"/>
       <geometry>
-        <cylinder length="0.018" radius="0.033"/>
+        <cylinder length="0.05" radius="0.0985"/>
       </geometry>
     </collision>

Commit message: changed lidar joint to fixed

File: urdf/warehouse_bot_sim.urdf.xacro (robot description, xacro)
@@ -136,5 +136,5 @@
     <axis xyz="0 0 1"/>
   </joint>
-  <joint name="base_link_to_laser_front" type="continuous">
+  <joint name="base_link_to_laser_front" type="fixed">
     <parent link="base_link"/>
     <child link="base_laser"/>

Commit message: updated robot urdf files

File: urdf/warehouse_bot_sim.urdf.xacro (robot description, xacro)
@@ -35,5 +35,5 @@
   </xacro:macro>
   <xacro:sensor_d435 parent="base_link" use_nominal_extrinsics="$(arg use_nominal_extrinsics)">
-    <origin xyz="0.25 0 0.254" rpy="0 0 0"/>
+    <origin xyz="0.19065 0 0.254" rpy="0 0 0"/>
   </xacro:sensor_d435>
   <xacro:caster name="caster_top_left">
