Commit message: Changed wheels to continuous

File: urdf/warehouse_bot_sim.urdf (robot description, URDF)
Before this commit: robot warehouse_bot, 5 links, 4 joints
Joints:
- joint base_link_to_laser_front: type fixed -> continuous
- joint wheel_right_joint: type fixed -> continuous

Commit message: Fixed incorrect frame definitions for wheels

File: urdf/warehouse_bot_sim.urdf (robot description, URDF)
Before this commit: robot warehouse_bot, 9 links, 8 joints
Links:
- link base_laser: mass None -> 0.003
- link base_link: mass 550 -> 20
- link wheel_left_link: geometry collision cylinder length=0.05 radius=0.0985; visual mesh filename=package://warehousebot_simulation/meshes/left_wheel.stl scale=0.01 0.01 0.01
- link wheel_right_link: geometry collision cylinder length=0.05 radius=0.0985; visual mesh filename=package://warehousebot_simulation/meshes/right_wheel.stl scale=0.01 0.01 0.01
Joints:
- joint base_link_to_laser_front: type continuous -> fixed
- joint wheel_left_joint: origin xyz=0 0.159974 0.0485 rpy=1.57 0 0 -> xyz=0 0.159974 0.0485 rpy=-1.57 0 0
- joint wheel_right_joint: origin xyz=0 -0.159974 0.0485 rpy=1.57 0 0 -> xyz=0 -0.159974 0.0485 rpy=-1.57 0 0

File: urdf/warehouse_bot_sim.urdf.xacro (robot description, xacro)
@@ -127,5 +127,5 @@
     <parent link="base_link"/>
     <child link="wheel_left_link"/>
-    <origin xyz="0 0.159974 0.0485" rpy="1.57 0 0"/>
+    <origin xyz="0 0.159974 0.0485" rpy="-1.57 0 0"/>
     <axis xyz="0 0 1"/>
   </joint>
@@ -133,5 +133,5 @@
     <parent link="base_link"/>
     <child link="wheel_right_link"/>
-    <origin xyz="0 -0.159974 0.0485" rpy="1.57 0 0"/>
+    <origin xyz="0 -0.159974 0.0485" rpy="-1.57 0 0"/>
     <axis xyz="0 0 1"/>
   </joint>

Commit message: Added in depth camera into robot urdf

File: urdf/warehouse_bot_sim.urdf (robot description, URDF)
Before this commit: robot warehouse_bot, 9 links, 8 joints
Links:
- added link camera_bottom_screw_frame
- added link camera_color_frame
- added link camera_color_optical_frame
- added link camera_depth_frame
- added link camera_depth_optical_frame
- added link camera_infra1_frame
- added link camera_infra1_optical_frame
- added link camera_infra2_frame
- added link camera_infra2_optical_frame
- added link camera_link; visual mesh filename=package://warehousebot_simulation/meshes/d435.dae
Joints:
- added joint camera_color_joint: type fixed, parent camera_link, child camera_color_frame, origin xyz=0 0.015 0 rpy=0 0 0
- added joint camera_color_optical_joint: type fixed, parent camera_color_frame, child camera_color_optical_frame, origin xyz=0 0 0 rpy=-1.5707963267948966 0 -1.5707963267948966
- added joint camera_depth_joint: type fixed, parent camera_link, child camera_depth_frame, origin xyz=0 0 0 rpy=0 0 0
- added joint camera_depth_optical_joint: type fixed, parent camera_depth_frame, child camera_depth_optical_frame, origin xyz=0 0 0 rpy=-1.5707963267948966 0 -1.5707963267948966
- added joint camera_infra1_joint: type fixed, parent camera_link, child camera_infra1_frame, origin xyz=0 0.0 0 rpy=0 0 0
- added joint camera_infra1_optical_joint: type fixed, parent camera_infra1_frame, child camera_infra1_optical_frame, origin xyz=0 0 0 rpy=-1.5707963267948966 0 -1.5707963267948966
- added joint camera_infra2_joint: type fixed, parent camera_link, child camera_infra2_frame, origin xyz=0 -0.05 0 rpy=0 0 0
- added joint camera_infra2_optical_joint: type fixed, parent camera_infra2_frame, child camera_infra2_optical_frame, origin xyz=0 0 0 rpy=-1.5707963267948966 0 -1.5707963267948966
- added joint camera_joint: type fixed, parent base_link, child camera_bottom_screw_frame, origin xyz=0.25 0 0.254 rpy=0 0 0
- added joint camera_link_joint: type fixed, parent camera_bottom_screw_frame, child camera_link, origin xyz=0.010600000000000002 0.0175 0.0125 rpy=0 0 0

File: urdf/warehouse_bot_sim.urdf.xacro (robot description, xacro)
@@ -3,4 +3,6 @@
   xmlns:xacro="http://ros.org/wiki/xacro">
   <xacro:include filename="$(find warehousebot_simulation)/urdf/warehouse_bot_sim.gazebo.xacro"/>
+  <xacro:include filename="$(find warehousebot_simulation)/urdf/_d435.urdf.xacro" />
+  <xacro:arg name="use_nominal_extrinsics" default="true"/>
   <xacro:macro name="caster" params="name *origin">
     <link name="${name}_link">
@@ -32,4 +34,7 @@
     </joint>
   </xacro:macro>
+  <xacro:sensor_d435 parent="base_link" use_nominal_extrinsics="$(arg use_nominal_extrinsics)">
+    <origin xyz="0.25 0 0.254" rpy="0 0 0"/>
+  </xacro:sensor_d435>
   <xacro:caster name="caster_top_left">
     <origin xyz="0.16 0.16 -0.035" rpy="0.0 0.0 0.0"/>

Commit message: updated generated files

File: urdf/warehouse_bot_sim.urdf (robot description, URDF)
Before this commit: robot warehouse_bot, 19 links, 18 joints
Joints:
- joint camera_joint: origin xyz=0.25 0 0.254 rpy=0 0 0 -> xyz=0.19065 0 0.254 rpy=0 0 0
