Commit message: Added in imu

File: urdf/_d435.gazebo.xacro (robot description, xacro)
@@ -1,9 +1,82 @@
 <?xml version="1.0"?>
-<!-- License: Apache 2.0. See LICENSE file in root directory. Copyright(c) 2017 PAL Robotics, S.L. All Rights Reserved This is the Gazebo URDF model for the Intel RealSense D435 camera -->
+<!-- License: Apache 2.0. See LICENSE file in root directory. Copyright(c) 2017 PAL Robotics, S.L.
+All Rights Reserved This is the Gazebo URDF model for the Intel RealSense D435 camera -->
 <robot xmlns:xacro="http://ros.org/wiki/xacro">
-  <xacro:macro name="gazebo_d435" params="camera_name reference_link topics_ns depth_optical_frame color_optical_frame infrared1_optical_frame infrared2_optical_frame image_width image_height">
+  <xacro:macro name="gazebo_d435"
+    params="camera_name reference_link topics_ns depth_optical_frame color_optical_frame infrared1_optical_frame infrared2_optical_frame image_width image_height">
     <!-- Load parameters to model's main link-->
-    <xacro:property name="deg_to_rad" value="0.01745329251994329577"/>
-    <gazebo reference="${camera_name}_color_frame">
+    <xacro:property
+      name="deg_to_rad" value="0.01745329251994329577" />
+    <gazebo
+      reference="${camera_name}_imu_optical_frame">
+      <sensor name="imu_sensor" type="imu">
+        <plugin filename="libgazebo_ros_imu_sensor.so" name="imu_plugin">
+          <ros>
+            <remapping>~/out:=imu/data</remapping>
+          </ros>
+          <initial_orientation_as_reference>false</initial_orientation_as_reference>
+        </plugin>
+        <always_on>true</always_on>
+        <update_rate>100</update_rate>
+        <visualize>true</visualize>
+        <frameName>camera_imu_optical_frame</frameName>
+        <imu>
+          <angular_velocity>
+            <x>
+              <noise type="gaussian">
+                <mean>0.0</mean>
+                <stddev>2e-4</stddev>
+                <bias_mean>0.0000075</bias_mean>
+                <bias_stddev>0.0000008</bias_stddev>
+              </noise>
+            </x>
+            <y>
+              <noise type="gaussian">
+                <mean>0.0</mean>
+                <stddev>2e-4</stddev>
+                <bias_mean>0.0000075</bias_mean>
+                <bias_stddev>0.0000008</bias_stddev>
+              </noise>
+            </y>
+            <z>
+              <noise type="gaussian">
+                <mean>0.0</mean>
+                <stddev>2e-4</stddev>
+                <bias_mean>0.0000075</bias_mean>
+                <bias_stddev>0.0000008</bias_stddev>
+              </noise>
+            </z>
+          </angular_velocity>
+          <linear_acceleration>
+            <x>
+              <noise type="gaussian">
+                <mean>0.0</mean>
+                <stddev>1.7e-2</stddev>
+                <bias_mean>0.1</bias_mean>
+                <bias_stddev>0.001</bias_stddev>
+              </noise>
+            </x>
+            <y>
+              <noise type="gaussian">
+                <mean>0.0</mean>
+                <stddev>1.7e-2</stddev>
+                <bias_mean>0.1</bias_mean>
+                <bias_stddev>0.001</bias_stddev>
+              </noise>
+            </y>
+            <z>
+              <noise type="gaussian">
+                <mean>0.0</mean>
+                <stddev>1.7e-2</stddev>
+                <bias_mean>0.1</bias_mean>
+                <bias_stddev>0.001</bias_stddev>
+              </noise>
+            </z>
+          </linear_acceleration>
+        </imu>
+      </sensor>
+    </gazebo>
+    <gazebo
+      reference="${camera_name}_color_frame">
       <self_collide>0</self_collide>
       <enable_wind>0</enable_wind>
@@ -13,5 +86,6 @@
       <mu2>1</mu2>
       <fdir1>0 0 0</fdir1>
-      <!--<slip1>0</slip1> <slip2>0</slip2>-->
+      <!--<slip1>0</slip1>
+      <slip2>0</slip2>-->
       <kp>1e+13</kp>
       <kd>1</kd>
@@ -47,8 +121,10 @@
       <mu2>1</mu2>
       <fdir1>0 0 0</fdir1>
-      <!--<slip1>0</slip1> <slip2>0</slip2>-->
+      <!--<slip1>0</slip1>
+      <slip2>0</slip2>-->
       <kp>1e+13</kp>
       <kd>1</kd>
-      <!--<max_vel>0.01</max_vel> <min_depth>0</min_depth>-->
+      <!--<max_vel>0.01</max_vel>
+      <min_depth>0</min_depth>-->
       <sensor name="${camera_name}ired1" type="camera">
         <camera name="${camera_name}">
@@ -116,7 +192,5 @@
         <visualize>0</visualize>
       </sensor>
-    </gazebo>
-    i
-    <gazebo>
+    </gazebo> i <gazebo>
       <plugin name="${topics_ns}" filename="libwarehousebot_simulation.so">
         <prefix>${camera_name}</prefix>

File: urdf/_d435.urdf.xacro (robot description, xacro)
@@ -69,4 +69,11 @@
       </visual>
     </link>
+     <!-- frames for imu -->
+    <link name="${name}_imu_optical_frame" />
+    <joint name="${name}_imu_joint" type="fixed">
+      <origin xyz = "-0.01174 -0.00552 0.0051" rpy = "0 0 0" />
+      <parent link="${name}_link" />
+      <child link="${name}_imu_optical_frame" />
+    </joint>
     <!-- Use the nominal extrinsics between camera frames if the calibrated extrinsics aren't being published. e.g. running the device in simulation  -->
     <xacro:if value="${use_nominal_extrinsics}">

File: urdf/warehouse_bot_sim.gazebo.xacro (robot description, xacro)
@@ -114,5 +114,5 @@
       <!-- output -->
       <publish_odom>true</publish_odom>
-      <publish_odom_tf>true</publish_odom_tf>
+      <publish_odom_tf>false</publish_odom_tf>
       <publish_wheel_tf>false</publish_wheel_tf>
       <odometry_topic>odom</odometry_topic>

File: urdf/warehouse_bot_sim.urdf (robot description, URDF)
Before this commit: robot warehouse_bot, 19 links, 18 joints
Links:
- added link camera_imu_optical_frame
Joints:
- added joint camera_imu_joint: type fixed, parent camera_link, child camera_imu_optical_frame, origin xyz=-0.01174 -0.00552 0.0051 rpy=0 0 0
